File: so5cw-band-decoder/so5cw-band-decoder.kicad_sch (KiCad schematic)
At the start: 136 parts, among them J1 DA15_Receptacle, J2 AudioJack3_SwitchTR, J3 Barrel_Jack_MountingPin, J4 RJ45, K1 TIANBO-HJR-4102-L, K10 TIANBO-HJR-4102-L, K11 TIANBO-HJR-4102-L, K12 TIANBO-HJR-4102-L, K2 TIANBO-HJR-4102-L, K3 TIANBO-HJR-4102-L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

Commit message: Rearrange parts and route the critical connections. Needs cleanup.
Parts:
- renumbered K8 to K10, K10 to K11, K9 to K8, K11 to K9
Connections:
- net R1A: now also R6.2; no longer R1.2
- net R1B: now also R5.2; no longer R2.2
- net R1C: now also R4.2; no longer R3.2
- net R1D: now also R3.2; no longer R4.2
- net R1E: now also R2.2; no longer R5.2
- net R1F: now also R1.2; no longer R6.2
- net R2A: now also R12.2; no longer R7.2
- net R2B: now also R11.2; no longer R8.2
- net R2C: now also R10.2; no longer R9.2
- net R2D: now also R9.2; no longer R10.2
- net R2E: now also R8.2; no longer R11.2
- net R2F: now also R7.2; no longer R12.2
Changed lines of the file:
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@@
     (effects (font (size 1.27 1.27)) (justify left bottom))
   )
-  (label "R1E" (at 19.05 151.13 0) (fields_autoplaced)
+  (label "R1B" (at 19.05 151.13 0) (fields_autoplaced)
     (effects (font (size 1.27 1.27)) (justify left bottom))
   )
@@
     (effects (font (size 1.27 1.27)) (justify left bottom))
   )
-  (label "R2A" (at 19.05 156.21 0) (fields_autoplaced)
+  (label "R2F" (at 19.05 156.21 0) (fields_autoplaced)
     (effects (font (size 1.27 1.27)) (justify left bottom))
   )
@@
     (effects (font (size 1.27 1.27)) (justify left bottom))
   )
-  (label "R2F" (at 19.05 168.91 0) (fields_autoplaced)
+  (label "R2A" (at 19.05 168.91 0) (fields_autoplaced)
     (effects (font (size 1.27 1.27)) (justify left bottom))
   )
-  (label "R2B" (at 19.05 158.75 0) (fields_autoplaced)
+  (label "R2E" (at 19.05 158.75 0) (fields_autoplaced)
     (effects (font (size 1.27 1.27)) (justify left bottom))
   )
@@
     (effects (font (size 1.27 1.27)) (justify left bottom))
   )
-  (label "R1C" (at 19.05 146.05 0) (fields_autoplaced)
+  (label "R1D" (at 19.05 146.05 0) (fields_autoplaced)
     (effects (font (size 1.27 1.27)) (justify left bottom))
   )
@@
     (effects (font (size 1.27 1.27)) (justify left bottom))
   )
-  (label "R1A" (at 19.05 140.97 0) (fields_autoplaced)
+  (label "R1F" (at 19.05 140.97 0) (fields_autoplaced)
     (effects (font (size 1.27 1.27)) (justify left bottom))
   )
@@
     (effects (font (size 1.27 1.27)) (justify left bottom))
   )
-  (label "R2C" (at 19.05 161.29 0) (fields_autoplaced)
+  (label "R2D" (at 19.05 161.29 0) (fields_autoplaced)
     (effects (font (size 1.27 1.27)) (justify left bottom))
   )
@@
     (effects (font (size 1.27 1.27)) (justify left bottom))
   )
-  (label "R2D" (at 19.05 163.83 0) (fields_autoplaced)
+  (label "R2C" (at 19.05 163.83 0) (fields_autoplaced)
     (effects (font (size 1.27 1.27)) (justify left bottom))
   )
@@
     (effects (font (size 1.27 1.27)) (justify left bottom))
   )
-  (label "R2E" (at 19.05 166.37 0) (fields_autoplaced)
+  (label "R2B" (at 19.05 166.37 0) (fields_autoplaced)
     (effects (font (size 1.27 1.27)) (justify left bottom))
   )
@@
     (effects (font (size 1.27 1.27)) (justify left bottom))
   )
-  (label "R1D" (at 19.05 148.59 0) (fields_autoplaced)
+  (label "R1C" (at 19.05 148.59 0) (fields_autoplaced)
     (effects (font (size 1.27 1.27)) (justify left bottom))
   )
@@
     (effects (font (size 1.27 1.27)) (justify left bottom))
   )
-  (label "R1B" (at 19.05 143.51 0) (fields_autoplaced)
+  (label "R1E" (at 19.05 143.51 0) (fields_autoplaced)
     (effects (font (size 1.27 1.27)) (justify left bottom))
   )
@@
     (effects (font (size 1.27 1.27)) (justify left bottom))
   )
-  (label "R1F" (at 19.05 153.67 0) (fields_autoplaced)
+  (label "R1A" (at 19.05 153.67 0) (fields_autoplaced)
     (effects (font (size 1.27 1.27)) (justify left bottom))
   )
@@
   (symbol (lib_id "Relay:TIANBO-HJR-4102-L") (at 269.24 76.2 0) (unit 1)
     (in_bom yes) (on_board yes) (dnp no) (fields_autoplaced)
-    (property "Reference" "K11" (at 280.67 74.93 0)
+    (property "Reference" "K9" (at 280.67 76.2 0)
       (effects (font (size 1.27 1.27)) (justify left))
     )
@@
       (project "so5cw-band-decoder"
         (path "/a618e2d6-97dd-4ea5-8871-d9a3161419a9"
-          (reference "K11") (unit 1)
+          (reference "K9") (unit 1)
         )
       )
@@
   (symbol (lib_id "Relay:TIANBO-HJR-4102-L") (at 234.95 99.06 0) (unit 1)
     (in_bom yes) (on_board yes) (dnp no) (fields_autoplaced)
-    (property "Reference" "K10" (at 246.38 97.79 0)
+    (property "Reference" "K11" (at 246.38 99.06 0)
       (effects (font (size 1.27 1.27)) (justify left))
     )
@@
       (project "so5cw-band-decoder"
         (path "/a618e2d6-97dd-4ea5-8871-d9a3161419a9"
-          (reference "K10") (unit 1)
+          (reference "K11") (unit 1)
         )
       )
@@
   (symbol (lib_id "Relay:TIANBO-HJR-4102-L") (at 234.95 76.2 0) (unit 1)
     (in_bom yes) (on_board yes) (dnp no) (fields_autoplaced)
-    (property "Reference" "K9" (at 246.38 74.93 0)
+    (property "Reference" "K8" (at 246.38 76.2 0)
       (effects (font (size 1.27 1.27)) (justify left))
     )
@@
       (project "so5cw-band-decoder"
         (path "/a618e2d6-97dd-4ea5-8871-d9a3161419a9"
-          (reference "K9") (unit 1)
+          (reference "K8") (unit 1)
         )
       )
@@
   (symbol (lib_id "Relay:TIANBO-HJR-4102-L") (at 200.66 99.06 0) (unit 1)
     (in_bom yes) (on_board yes) (dnp no)
-    (property "Reference" "K8" (at 212.09 97.79 0)
+    (property "Reference" "K10" (at 212.09 97.79 0)
       (effects (font (size 1.27 1.27)) (justify left))
     )
@@
       (project "so5cw-band-decoder"
         (path "/a618e2d6-97dd-4ea5-8871-d9a3161419a9"
-          (reference "K8") (unit 1)
+          (reference "K10") (unit 1)
         )
       )

Commit message: some more routing, add buzzer, heatsink for 5V reg, etc.
Parts:
- removed J3: Barrel_Jack_MountingPin, Connector_BarrelJack:BarrelJack_CLIFF_FC681465S_SMT_Horizontal, symbol Connector:Barrel_Jack_MountingPin
- added BZ1: Buzzer, so5cw-band-decoder-components:Buzzer_12x9.5RM6.5, symbol Device:Buzzer
- added C47: 47u, Capacitor_SMD:CP_Elec_6.3x7.7, symbol Device:C_Polarized_Small
- added C48, C49: 100n, Capacitor_SMD:C_0603_1608Metric_Pad1.08x0.95mm_HandSolder, symbol Device:C
- added FID1: KiCad Logo, Symbol:KiCad-Logo2_6mm_SilkScreen, symbol Mechanical:Fiducial
- added HS1: Heatsink_Pad, Heatsink:Heatsink_Fischer_SK104-STC-STIC_35x13mm_2xDrill2.5mm, symbol Mechanical:Heatsink_Pad
- added J3: Barrel_Jack, Connector_BarrelJack:BarrelJack_CLIFF_FC681465S_SMT_Horizontal, symbol Connector:Barrel_Jack
- added J5: Conn_01x02_Pin, Connector_PinHeader_2.54mm:PinHeader_1x02_P2.54mm_Vertical, symbol Connector:Conn_01x02_Pin
- added TP1, TP2, TP3, TP4, TP5, TP6, TP7, TP8, TP9: TestPoint, TestPoint:TestPoint_THTPad_1.0x1.0mm_Drill0.5mm, symbol Connector:TestPoint
Connections:
- net +12V: now also C48.1, C49.1, J5.2 (Pin_2), TP6.1
- net +5V: now also C47.1, TP5.1
- net GND: now also BZ1.2 (-), C47.2, C48.2, C49.2, HS1.1, J3.2, J5.1 (Pin_1)
- net R1_BAND: now also J4.1, R16.1; no longer J4.7, R15.1
- net R1_TX: now also J4.7, R14.1; no longer J4.1, R13.1
- net R2_BAND: now also J4.2, R15.1; no longer J4.8, R16.1
- net R2_TX: now also J4.8, R13.1; no longer J4.2, R14.1
- net UART_RX: now also TP7.1
- net UART_TX: now also TP8.1
- net at C29.1, J2.T, Q1.1 (G)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: now also TP9.1
- net at R15.2, U1.31 (GPIO26_ADC0): now also TP3.1
- net at R14.2, U1.29 (GPIO22): now also TP2.1
- net at C33.1, L13.1: now also J3.1
- net at R13.2, U1.27 (GPIO21): now also TP1.1
- net at R16.2, U1.32 (GPIO27_ADC1): now also TP4.1
- net BUZZER: now reaches U1.5 (GPIO3)
- net BUZZER: now also BZ1.1 (+)
Other:
- note added: "PCB cut for case TEKO 222"
- moved on the sheet: J4, R13, R14, R15, R16
